Commit message: first commit

File: velodyne_description/urdf/VLP-16.urdf.xacro (robot description, xacro)
@@ -2,5 +2,5 @@
 <robot xmlns:xacro="http://www.ros.org/wiki/xacro" name="VLP-16">
   <xacro:property name="M_PI" value="3.1415926535897931" />
-  <xacro:macro name="VLP-16" params="*origin parent:=base_link name:=velodyne topic:=/velodyne_points hz:=10 lasers:=16 samples:=1875 collision_range:=0.3 min_range:=0.9 max_range:=130.0 noise:=0.008 min_angle:=-${M_PI} max_angle:=${M_PI}">
+  <xacro:macro name="VLP-16" params="*origin parent:=base_link name:=velodyne topic:=/velodyne_points hz:=10 lasers:=16 samples:=1875 collision_range:=0.3 min_range:=0.9 max_range:=130.0 noise:=0.008 min_angle:=-${M_PI} max_angle:=${M_PI} vehicle_name:=vehicle">
     <joint name="${name}_base_mount_joint" type="fixed">
       <xacro:insert_block name="origin" />
@@ -82,6 +82,6 @@
         </ray>
         <plugin name="gazebo_ros_laser_controller" filename="libgazebo_ros_velodyne_laser.so">
-          <topicName>${topic}</topicName>
-          <frameName>/${name}</frameName>
+	  <topicName>${name}/${topic}</topicName>
+	  <frameName>${vehicle_name}/${name}</frameName>
           <min_range>${min_range}</min_range>
           <max_range>${max_range}</max_range>

File: velodyne_description/urdf/example.urdf.xacro (robot description, xacro)
@@ -2,12 +2,13 @@
 <robot xmlns:xacro="http://www.ros.org/wiki/xacro" name="example">
   <!-- Base Footprint -->
-  <link name="base_footprint" />
+  <!--  <link name="vehicle/base_footprint" /> -->
+  <link name="vehicle/base_link" />
   <!-- Base Link -->
-  <joint name="footprint" type="fixed" >
-   <parent link="base_footprint" />
-    <child link="base_link" />
-    <origin xyz="0 0 0.05" rpy="0 0 0" />
+  <!--  <joint name="footprint" type="fixed" >
+    <parent link="base_footprint" />
+    <child link="vehicle/velodyne_base" />
+    <origin xyz="0 0 1.45" rpy="0 0 0" />
   </joint>
-  <link name="base_link" >
+  <link name="vehicle/velodyne_base" >
     <visual>
       <geometry>
@@ -27,12 +28,12 @@
                izz="3.0" />
     </inertial>
-  </link>
+  </link> -->
   <xacro:include filename="$(find velodyne_description)/urdf/VLP-16.urdf.xacro"/>
-  <VLP-16 parent="base_link" name="velodyne" topic="/velodyne_points" hz="10" samples="440">
-    <origin xyz="0 0 0.4" rpy="0 0 0" />
+  <VLP-16 parent="vehicle/base_link" name="velodyne" topic="vehicle/velodyne_points" hz="10" samples="440">
+    <origin xyz="0 0 1.7" rpy="0 0 0" />
   </VLP-16>
-  <xacro:include filename="$(find velodyne_description)/urdf/HDL-32E.urdf.xacro"/>
+  <!--  <xacro:include filename="$(find velodyne_description)/urdf/HDL-32E.urdf.xacro"/>
   <HDL-32E parent="base_link" name="velodyne2" topic="/velodyne_points2" hz="10" samples="220">
     <origin xyz="0 0 0.6" rpy="0 0 0" />
-  </HDL-32E>
+  </HDL-32E> -->
 </robot>
